Commit message: feat: harden generalized grasp scene safety

File: ros2_ws/src/strawberry_sim/urdf/dynamic_attachments.xacro (robot description, xacro)
@@ -12,3 +12,17 @@
     </plugin>
   </xacro:macro>
+  <xacro:macro name="strawberry_stem_attachment" params="target_id">
+    <!-- Generalized-scene fruit must remain plant-supported before grasp.
+         panda_link0 is fixed to the world, so this models a stationary stem
+         without adding a runtime truth or control input. -->
+    <plugin filename="gz-sim-detachable-joint-system"
+            name="gz::sim::systems::DetachableJoint">
+      <parent_link>panda_link0</parent_link>
+      <child_model>strawberry_${target_id}</child_model>
+      <child_link>fruit_link</child_link>
+      <attach_topic>/strawberry/sim/fruit_${target_id}/stem_attach</attach_topic>
+      <detach_topic>/strawberry/sim/fruit_${target_id}/stem_detach</detach_topic>
+      <output_topic>/strawberry/sim/fruit_${target_id}/stem_attached</output_topic>
+    </plugin>
+  </xacro:macro>
 </robot>

File: ros2_ws/src/strawberry_sim/urdf/panda_gz.urdf.xacro (robot description, xacro)
@@ -4,4 +4,5 @@
              default="$(find strawberry_sim)/config/panda_initial_positions.yaml"/>
   <xacro:arg name="enable_attachment" default="false"/>
+  <xacro:arg name="enable_stem_attachment" default="false"/>
   <xacro:arg name="fruit_attachment_count" default="3"/>
   <xacro:arg name="camera_mount" default="fixed"/>
@@ -301,4 +302,15 @@
       <xacro:if value="${int('$(arg fruit_attachment_count)') >= 8}"><xacro:strawberry_attachment target_id="8"/></xacro:if>
       <xacro:if value="${int('$(arg fruit_attachment_count)') >= 9}"><xacro:strawberry_attachment target_id="9"/></xacro:if>
+      <xacro:if value="$(arg enable_stem_attachment)">
+        <xacro:strawberry_stem_attachment target_id="1"/>
+        <xacro:if value="${int('$(arg fruit_attachment_count)') >= 2}"><xacro:strawberry_stem_attachment target_id="2"/></xacro:if>
+        <xacro:if value="${int('$(arg fruit_attachment_count)') >= 3}"><xacro:strawberry_stem_attachment target_id="3"/></xacro:if>
+        <xacro:if value="${int('$(arg fruit_attachment_count)') >= 4}"><xacro:strawberry_stem_attachment target_id="4"/></xacro:if>
+        <xacro:if value="${int('$(arg fruit_attachment_count)') >= 5}"><xacro:strawberry_stem_attachment target_id="5"/></xacro:if>
+        <xacro:if value="${int('$(arg fruit_attachment_count)') >= 6}"><xacro:strawberry_stem_attachment target_id="6"/></xacro:if>
+        <xacro:if value="${int('$(arg fruit_attachment_count)') >= 7}"><xacro:strawberry_stem_attachment target_id="7"/></xacro:if>
+        <xacro:if value="${int('$(arg fruit_attachment_count)') >= 8}"><xacro:strawberry_stem_attachment target_id="8"/></xacro:if>
+        <xacro:if value="${int('$(arg fruit_attachment_count)') >= 9}"><xacro:strawberry_stem_attachment target_id="9"/></xacro:if>
+      </xacro:if>
     </xacro:if>
   </gazebo>
