Commit message: Add validated field-v3 perception pick

File: ros2_ws/src/strawberry_sim/urdf/panda_gz.urdf.xacro (robot description, xacro)
@@ -242,5 +242,9 @@
       <state_interface name="velocity"/>
     </joint>
-    <joint name="panda_finger_joint2">
+    <!-- Disable ros2_control's mimic activation for this hardware interface:
+         DART does not apply the URDF mimic constraint, so a second controller
+         must command the physical simulation joint explicitly. -->
+    <joint name="panda_finger_joint2" mimic="false">
+      <command_interface name="position"/>
       <state_interface name="position"><param name="initial_value">0.04</param></state_interface>
       <state_interface name="velocity"/>

Commit message: feat: prove safe partial multi-target harvest

File: ros2_ws/src/strawberry_sim/urdf/panda_gz.urdf.xacro (robot description, xacro)
@@ -122,5 +122,7 @@
       <parent link="panda_link0"/>
       <child link="strawberry_base_camera_mast"/>
-      <origin xyz="-0.10 -0.42 0.05" rpy="0 0 0"/>
+      <!-- Lateral offset keeps the verified ready arm out of the plant-core
+           image region while preserving the complete conservative workspace. -->
+      <origin xyz="-0.35 0.45 0.05" rpy="0 0 0"/>
     </joint>
     <gazebo reference="panda_base_camera_mast_joint">
@@ -134,5 +136,5 @@
         parent_link="strawberry_base_camera_mast"
         xyz="0 0 1.00"
-        rpy="0 0.599 0.611"
+        rpy="0 0.543 -0.480"
         topic="/camera/base"
         sensor_name="base_rgbd"

Commit message: feat: gate generalized scenes on visual observability

File: ros2_ws/src/strawberry_sim/urdf/panda_gz.urdf.xacro (robot description, xacro)
@@ -7,4 +7,7 @@
   <xacro:arg name="fruit_attachment_count" default="3"/>
   <xacro:arg name="camera_mount" default="fixed"/>
+  <xacro:arg name="base_camera_mast_xyz" default="-0.35 0.45 0.05"/>
+  <xacro:arg name="base_camera_xyz" default="0 0 1.00"/>
+  <xacro:arg name="base_camera_rpy" default="0 0.543 -0.480"/>
   <xacro:property name="initial_positions"
                   value="${xacro.load_yaml('$(arg initial_positions_file)')['initial_positions']}"/>
@@ -124,5 +127,5 @@
       <!-- Lateral offset keeps the verified ready arm out of the plant-core
            image region while preserving the complete conservative workspace. -->
-      <origin xyz="-0.35 0.45 0.05" rpy="0 0 0"/>
+      <origin xyz="$(arg base_camera_mast_xyz)" rpy="0 0 0"/>
     </joint>
     <gazebo reference="panda_base_camera_mast_joint">
@@ -135,6 +138,6 @@
         optical_joint_name="strawberry_base_camera_optical_joint"
         parent_link="strawberry_base_camera_mast"
-        xyz="0 0 1.00"
-        rpy="0 0.543 -0.480"
+        xyz="$(arg base_camera_xyz)"
+        rpy="$(arg base_camera_rpy)"
         topic="/camera/base"
         sensor_name="base_rgbd"

Commit message: feat: hybrid control - effort gravity compensation j1-j6, position j7
v19 receipt: effort-mode integral gravity compensation holds joints
1-6 rock solid (<=0.001 rad per 0.4s) but joint7's tiny wrist-roll
inertia saturates the plugin's effort velocity clamp regardless of
gains (four variants, identical +/-2.871 bang-bang). Split the arm:
j1-j6 stay on panda_arm_controller (effort JTC, p300/p60, i150/40);
joint7 moves to a new single-joint panda_wrist_roll_controller on the
position interface that tracked it perfectly in v9-v11.

Backend _split_arm_goal divides every 7-joint goal into a 6-joint arm
goal and a 1-joint wrist goal with identical timing; both action
results must succeed. URDF, controllers.yaml, launch spawners and
contract tests updated; full regression green (854 pure / 228
manipulation / 119 sim / 145 bringup).

File: ros2_ws/src/strawberry_sim/urdf/panda_gz.urdf.xacro (robot description, xacro)
@@ -250,5 +250,14 @@
     <xacro:arm_control_joint name="panda_joint5"/>
     <xacro:arm_control_joint name="panda_joint6"/>
-    <xacro:arm_control_joint name="panda_joint7"/>
+    <!-- joint7 runs its own position-interface JTC (hybrid control): its tiny
+         inertia saturates the effort path's velocity clamp in one 100 Hz cycle
+         for any nonzero torque (v12-v19, receipt v19_findings_receipt.json). -->
+    <joint name="panda_joint7">
+      <command_interface name="position"/>
+      <state_interface name="position">
+        <param name="initial_value">${initial_positions["panda_joint7"]}</param>
+      </state_interface>
+      <state_interface name="velocity"/>
+    </joint>
     <joint name="panda_finger_joint1">
       <command_interface name="position"/>

Commit message: feat: plan A - position-interface baseline with zero-velocity window
v20 receipt: the hybrid split worked for joint7 (position controller,
3/3 goals) but the effort path injects velocity kicks on every joint,
scaled by inverse inertia (j4 kicked 0.09 rad at goal boundaries AND
mid-goal; position mode never kicks). Per user decision, revert the
arm to the position interface (v10 baseline) for all seven joints and
remove the hybrid split.

The surviving position-interface goal-boundary kick (v9/v10) is now
guarded by a zero-velocity confirmation window: after any goal
terminal, _execute_joint_path withholds the next goal until every
reported joint velocity stays inside +/-0.05 rad/s for 3 consecutive
samples, bounded by a 2 s fail-closed timeout. Contract tests replaced
with the plan-A control contract.

File: ros2_ws/src/strawberry_sim/urdf/panda_gz.urdf.xacro (robot description, xacro)
@@ -233,9 +233,10 @@
     <xacro:macro name="arm_control_joint" params="name">
       <joint name="${name}">
-        <!-- Effort is the claimed command interface: the trajectory controller
-             runs closed-loop PID with velocity feedforward, which balances the
-             attached-fruit gravity torque at steady state (the position-only
-             velocity law could not: v9/v10 aborted at 0.0531 rad vs 0.05). -->
-        <command_interface name="effort"/>
+        <!-- Position interface (plan A, v20 receipt): the plugin's effort path
+             injects velocity kicks scaled by inverse inertia (j7 bang-bang at
+             the clamp, j4 kicked 0.09 rad); the position velocity law tracks
+             cleanly. The surviving goal-boundary kick is guarded by the
+             backend zero-velocity confirmation window. -->
+        <command_interface name="position"/>
         <state_interface name="position">
           <param name="initial_value">${initial_positions[name]}</param>
@@ -250,14 +251,5 @@
     <xacro:arm_control_joint name="panda_joint5"/>
     <xacro:arm_control_joint name="panda_joint6"/>
-    <!-- joint7 runs its own position-interface JTC (hybrid control): its tiny
-         inertia saturates the effort path's velocity clamp in one 100 Hz cycle
-         for any nonzero torque (v12-v19, receipt v19_findings_receipt.json). -->
-    <joint name="panda_joint7">
-      <command_interface name="position"/>
-      <state_interface name="position">
-        <param name="initial_value">${initial_positions["panda_joint7"]}</param>
-      </state_interface>
-      <state_interface name="velocity"/>
-    </joint>
+    <xacro:arm_control_joint name="panda_joint7"/>
     <joint name="panda_finger_joint1">
       <command_interface name="position"/>
@@ -287,8 +279,8 @@
            Measured bounds (seed 45504 probes): 1.0 tracks but sags under wrist
            payload near tolerance (v9/v10 aborts at 0.0531 vs 0.05); 3.0 sustains
-           a ~5.5 Hz +/-0.086 rad limit cycle at the frozen home pose and the arm
-           never settles (v11, commit 637135a, reverted). 1.0 stays until a
-           gravity-compensation or per-joint tuning change passes its own
-           oscillation gate. -->
+           a ~5.5 Hz +/-0.086 rad limit cycle at the frozen home pose (v11,
+           reverted); the effort-interface route (v12-v20) injects velocity
+           kicks scaled by inverse joint inertia. 1.0 stays; the goal-boundary
+           kick is guarded by the backend zero-velocity confirmation window. -->
       <position_proportional_gain>1.0</position_proportional_gain>
     </plugin>
